Commit message: fix: Critical fixes - URDF typo, sensor links, udev rules, documentation
- Fixed URDF line 226 typo (inertial → inertia) - CRITICAL bugfix
- Added missing sensor links to URDF:
  - imu_link (BNO055 IMU)
  - camera_link (RealSense D435)
  - elp_camera_link (ELP USB camera)
- Fixed CMakeLists.txt to only install existing directories
- Added udev rules to repository (config/udev/)
  - RPLidar: /dev/rplidar (persistent)
  - ELP camera: /dev/elp_camera (persistent)
  - RealSense D435: permissions configured
- Created comprehensive ELP camera documentation
- Updated README with complete 7-sensor hardware table

All critical issues from analysis resolved.
Repository ready for physical assembly!

File: ros2_ws/src/hoverbot_description/urdf/hoverbot.urdf (robot description, URDF)
Before this commit: robot hoverbot, 7 links, 6 joints
Links:
- added link camera_link, mass 0.072; collision box size=0.090 0.025 0.025; visual box size=0.090 0.025 0.025
- added link elp_camera_link, mass 0.050; collision box size=0.030 0.030 0.030; visual box size=0.030 0.030 0.030
- added link imu_link, mass 0.005; collision box size=0.025 0.025 0.010; visual box size=0.025 0.025 0.010
Joints:
- added joint camera_joint: type fixed, parent base_link, child camera_link, origin xyz=0.15 0.0 0.20 rpy=0 0 0
- added joint elp_camera_joint: type fixed, parent base_link, child elp_camera_link, origin xyz=0.15 0.05 0.20 rpy=0 0 0
- added joint imu_joint: type fixed, parent base_link, child imu_link, origin xyz=0.0 0.0 0.10 rpy=0 0 0
